Commit message: Modify robot urdf to be more accurate

File: description/lidar.xacro (robot description, xacro)
@@ -4,5 +4,5 @@
         <parent link="chassis"/>
         <child link="laser_frame"/>
-        <origin xyz="0.1 0.0 0.175" rpy="0.0 0.0 0.0"/>
+        <origin xyz="0.1 0.0 0.475" rpy="0.0 0.0 0.0"/>
     </joint>
     <link name="laser_frame">

File: description/robot_core.xacro (robot description, xacro)
@@ -5,6 +5,6 @@
         <color rgba="1 1 1 1"/>
     </material>
-    <material name="orange">
-        <color rgba="1 0.3 0.1 1"/>
+    <material name="brown">
+        <color rgba="0.34 0.14 0.07 1"/>
     </material>
     <material name="blue">
@@ -28,7 +28,7 @@
     <link name="chassis">
         <visual>
-            <origin xyz="0.15 0.0 0.075"/>
+            <origin xyz="0.15 0.0 0.225"/>
             <geometry>
-                <box size="0.3 0.3 0.15"/>
+                <box size="0.3 0.3 0.45"/>
             </geometry>
             <material name="white"/>
@@ -37,8 +37,8 @@
             <origin xyz="0.15 0.0 0.075"/>
             <geometry>
-                <box size="0.3 0.3 0.15"/>
+                <box size="0.3 0.3 0.45"/>
             </geometry>
         </collision>
-        <xacro:inertial_box mass="0.5" x="0.3" y="0.3" z="0.15">
+        <xacro:inertial_box mass="0.5" x="0.3" y="0.3" z="0.45">
             <origin xyz="0.15 0.0 0.075" rpy="0.0 0.0 0.0"/>
         </xacro:inertial_box>
@@ -57,5 +57,5 @@
         <visual>
             <geometry>
-                <cylinder radius="0.05" length="0.04"/>
+                <cylinder radius="0.035" length="0.04"/>
                 <material name="blue"/>
             </geometry>
@@ -63,8 +63,8 @@
         <collision>
             <geometry>
-                <cylinder radius="0.05" length="0.04"/>
+                <sphere radius="0.035" length="0.04"/>
             </geometry>
         </collision>
-        <xacro:inertial_cylinder mass="0.1" length="0.04" radius="0.05">
+        <xacro:inertial_cylinder mass="0.1" length="0.04" radius="0.035">
             <origin xyz="0.0 0.0 0.0" rpy="0.0 0.0 0.0"/>
         </xacro:inertial_cylinder>
@@ -83,5 +83,5 @@
         <visual>
             <geometry>
-                <cylinder radius="0.05" length="0.04"/>
+                <cylinder radius="0.035" length="0.04"/>
                 <material name="blue"/>
             </geometry>
@@ -89,8 +89,8 @@
         <collision>
             <geometry>
-                <cylinder radius="0.05" length="0.04"/>
+                <sphere radius="0.035" length="0.04"/>
             </geometry>
         </collision>
-        <xacro:inertial_cylinder mass="0.1" length="0.04" radius="0.05">
+        <xacro:inertial_cylinder mass="0.1" length="0.04" radius="0.035">
             <origin xyz="0.0 0.0 0.0" rpy="0.0 0.0 0.0"/>
         </xacro:inertial_cylinder>
