Commit message: Fix: put correct collision size

File: description/robot_core.xacro (robot description, xacro)
@@ -35,5 +35,5 @@
         </visual>
         <collision>
-            <origin xyz="0.15 0.0 0.075"/>
+            <origin xyz="0.15 0.0 0.225"/>
             <geometry>
                 <box size="0.3 0.3 0.45"/>
@@ -41,5 +41,5 @@
         </collision>
         <xacro:inertial_box mass="0.5" x="0.3" y="0.3" z="0.45">
-            <origin xyz="0.15 0.0 0.075" rpy="0.0 0.0 0.0"/>
+            <origin xyz="0.15 0.0 0.225" rpy="0.0 0.0 0.0"/>
         </xacro:inertial_box>
     </link>
@@ -63,5 +63,5 @@
         <collision>
             <geometry>
-                <sphere radius="0.035" length="0.04"/>
+                <sphere radius="0.035"/>
             </geometry>
         </collision>
@@ -89,5 +89,5 @@
         <collision>
             <geometry>
-                <sphere radius="0.035" length="0.04"/>
+                <sphere radius="0.035"/>
             </geometry>
         </collision>
@@ -108,5 +108,5 @@
         <visual>
             <geometry>
-                <sphere radius="0.05"/>
+                <sphere radius="0.035"/>
             </geometry>
             <material name="black"/>
@@ -114,5 +114,5 @@
         <collision>
             <geometry>
-                <sphere radius="0.05"/>
+                <sphere radius="0.035"/>
             </geometry>
         </collision>
